File: hardware/basic-inline-turbidimeter_main_board_v2.0.brd (EAGLE design)
At the start: 33.3 x 47 mm, 30 parts, among them IC1 MEGA8-AI

Commit message: minor updates
Parts:
- removed C12: 10uF, SparkFun:0603-CAP
- removed U$4: LMT86, open_source_turbidimeter:LMT86
- removed Y1: (no value), SparkFun:CRYSTAL-SMD-5X3
- added C9: 10uF, SparkFun:0603-CAP
- added FRAME1: FRAME-LETTER, SparkFun-Aesthetics:CREATIVE_COMMONS
- added Q1: (no value), SparkFun:CRYSTAL-SMD-5X3
- added T1: LMT86, open_source_turbidimeter:LMT86
- R1: value 10k -> 100k
- R2: value 1k -> 10k
- moved C4 1.37 mm to (6.35, 35.9)
- moved U$1 1.37 mm to (4.23, 42.5)
- moved U$3 1.37 mm to (29.2, 42.5)
- moved C6 1.37 mm to (6.35, 30.8)
- moved JP2 1.37 mm to (3.81, 12.1)
- moved JP6 1.37 mm to (6.35, 24.8)
- moved JP1 1.37 mm to (24.1, 9.02)
- moved JP5 1.37 mm to (26.7, 12.1)
- moved JP8 1.37 mm to (21.6, 9.02)
- moved PAD4 1.37 mm to (15.2, 38.1)
- moved U$5 1.37 mm to (29.2, 4.49)
- moved U$6 1.37 mm to (4.23, 4.49)
- moved *RTC 1.37 mm to (16.5, 27.0)
- moved C1 1.37 mm to (10.2, 24.4)
- moved C2 1.37 mm to (11.2, 14.0)
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Connections:
- net GND: now also C9.1, T1.1, T1.2; no longer C12.1, U$4.1, U$4.2
- net PC0: now also T1.3; no longer U$4.3
- net Q1: now also Q1.1; no longer Y1.1
- net Q2: now also Q1.3; no longer Y1.3
- net VCC: now also C9.2, T1.4, T1.5; no longer C12.2, U$4.4, U$4.5
Other:
- board text added: "Chris Kelley / AWQUA"
