File: hardware/basic-inline-turbidimeter_power_board.sch (EAGLE design)
At the start: 6 parts, among them IC1 LP298XS

Commit message: hardware updates
Parts:
- removed BOARD_OUT, LIPO_IN: (no value), adafruit:JST_2PIN-SMT-RA
- removed C1: OPT_0.01uF, SparkFun-Capacitors:CAP1206
- removed C5: 2.2uF, SparkFun-Capacitors:CAP1206
- removed IC1: LP298XS, adafruit:LP298XS
- added +OUT-, JP2: (no value), SparkFun-Connectors:M02PTH
- added 1UF, 2.2UF, OPT_10NF: (no value), SparkFun-Passives:CAP0603-CAP
- added C4: 4.7uF, SparkFun:CAP0402-CAP
- added D1: GREEN, SparkFun:LED0603
- added D11: RED, SparkFun:LED0603
- added D2: MBRA140, SparkFun-DiscreteSemi:MBRA140
- added JMP: (no value), SparkFun:M02PTH
- added JP7: LiPo Battery, SparkFun:M02-JST-2MM-SMT
- added R1: R330, SparkFun:RESISTOR0402-RES
- added R2K: 2K, SparkFun:RESISTOR0402-RES
- added R330: 330, SparkFun:RESISTOR0402-RES
- added U$2: LP2985, awqua_eagle_library:LP2985
- added U1: MCP73831, SparkFun:MCP73831
- C3: value 1.0uF -> 4.7uF; device SparkFun-Capacitors:CAP1206 -> SparkFun:CAP0402-CAP
Connections:
- removed net VOUT: BOARD_OUT.2, C5.1, IC1.VOUT
- new net N$2: D1.A, R1.2
- new net N$3: D11.A, R330.1
- new net N$4: +OUT-.1, 2.2UF.1, U$2.VOUT
- new net N$5: D2.A, JP2.2
- new net PROG: R2K.1, U1.PROG
- new net STAT: D11.C, R1.1, U1.STAT
- new net VIN: C3.1, D2.C, R330.2, U1.VIN
- net GND: now also +OUT-.2, 1UF.2, 2.2UF.2, C4.2, D1.C, JMP.1, JP2.1, JP7.1, OPT_10NF.2, R2K.2, U$2.GND, U1.VSS; no longer BOARD_OUT.1, C1.2, C5.2, IC1.GND, LIPO_IN.1
- net N$1: now also OPT_10NF.1, U$2.BYP; no longer C1.1, IC1.BYP
- net VCC: now also 1UF.1, C4.1, JMP.2, JP7.2, U$2.EN, U$2.VIN, U1.VBAT; no longer C3.1, IC1.EN, IC1.VIN, LIPO_IN.2
Other:
- note added: "0.1""
- note added: "3.3V Power Connection"
- note added: "3.7V Power Connection"
- note added: "INPUT"
- note added: "N. Seidle"
- note added: "Set (R2K) for 500mA charging"
- moved on the sheet: C3

Commit message: minor updates
Parts:
- removed C3: 4.7uF, SparkFun:CAP0402-CAP
- removed D2: MBRA140, SparkFun-DiscreteSemi:MBRA140
- added C12: 4.7uF, SparkFun:CAP0402-CAP
- added DS1: MBRA140, SparkFun-DiscreteSemi:MBRA140
- C10: value (none) -> 1uF
- C11: value (none) -> 2.2uF
- C14: value (none) -> 10nF (OPT)
- R5: value R330 -> 330
- renumbered 1UF to C10, 2.2UF to C11, C4 to C13, D1 to LG1, D11 to LR1, OPT_10NF to C14, R1 to R5, R2K to R3, R330 to R4, U$2 to VR1, U1 to BC1
Connections:
- net GND: now also C12.2; no longer C3.2
- net N$5: now also DS1.A; no longer D2.A
- net VIN: now also C12.1, DS1.C; no longer C3.1, D2.C
