File: hardware/basic-inline-turbidimeter_sensor_board_4led.brd (EAGLE design)
At the start: 44.5 x 20.3 mm, 15 parts

Commit message: minor updates
Parts:
- removed D5, D6: AL5809, diode:SOD123
- removed JP1: (no value), SparkFun-Connectors:1X06
- removed U$3: TSL230RDSMD, open_source_turbidimeter:TSL230RD
- added D3, D4: AL5809, diode:SOD123
- added FRAME1: FRAME-LETTER, SparkFun-Aesthetics:CREATIVE_COMMONS
- added HS1: (no value), SparkFun-Connectors:1X06
- added S1: TSL230RDSMD, open_source_turbidimeter:TSL230RD
- moved LED1 1.27 mm to (40.6, 15.2)
- moved LED2 1.27 mm to (3.81, 15.2)
- moved D1 1.27 mm to (8.89, 5.71)
- moved JP6 1.27 mm to (12.1, 6.35)
- moved JP2 1.27 mm to (9.53, 1.27)
- moved U$5 1.27 mm to (3.33, 1.91)
- moved C2 1.27 mm to (22.2, 14.6)
- moved D2 1.27 mm to (35.6, 5.08)
- moved JP5 1.27 mm to (12.1, 14.0)
- moved LED3 1.27 mm to (3.81, 8.26)
- moved LED4 1.27 mm to (40.6, 8.26)
Connections:
- net GND_2: now also HS1.GND, S1.GND, S1.S3; no longer JP1.GND, U$3.GND, U$3.S3
- net N$5: now also D4.C; no longer D6.C
- net N$7: now also D3.C; no longer D5.C
- net PC1_2: now also HS1.CTS, S1.OE; no longer JP1.CTS, U$3.OE
- net PD2_2: now also S1.OUT; no longer U$3.OUT
- net PD3_2: now also D3.A; no longer D5.A
- net PD4_2: now also D4.A; no longer D6.A
- net PD7_2: now also S1.S1; no longer U$3.S1
- net VCC_2: now also HS1.VCC, S1.S0, S1.S2, S1.VDD; no longer JP1.VCC, U$3.S0, U$3.S2, U$3.VDD
