File: hardware/basic-inline-turbidimeter_sensor_board_4led.sch (EAGLE design)
At the start: 14 parts

Commit message: minor updates
Parts:
- added FRAME1: FRAME-LETTER, SparkFun-Aesthetics:FRAME-LETTER
- renumbered D5 to D3, D6 to D4, JP1 to HS1, U$3 to S1
Other:
- note added: "Chris Kelley"
Changed lines of the file:
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@@
 <part name="LED3" library="SparkFun-LED" deviceset="LED" device="5MM"/>
 <part name="LED4" library="SparkFun-LED" deviceset="LED" device="5MM"/>
-<part name="U$3" library="open_source_turbidimeter" deviceset="TSL230RD" device="SMD"/>
+<part name="S1" library="open_source_turbidimeter" deviceset="TSL230RD" device="SMD"/>
 <part name="C2" library="SparkFun-Capacitors" deviceset="CAP" device="0805" value="100n"/>
-<part name="JP1" library="SparkFun-Connectors" deviceset="M06" device="SIP"/>
+<part name="HS1" library="SparkFun-Connectors" deviceset="M06" device="SIP"/>
 <part name="JP5" library="SparkFun-Connectors" deviceset="M03" device="PTH"/>
 <part name="JP6" library="SparkFun-Connectors" deviceset="M03" device="PTH"/>
 <part name="GND1" library="SparkFun" deviceset="GND" device=""/>
-<part name="D5" library="diode" deviceset="DIODE-" device="SOD123" value="AL5809"/>
-<part name="D6" library="diode" deviceset="DIODE-" device="SOD123" value="AL5809"/>
+<part name="D3" library="diode" deviceset="DIODE-" device="SOD123" value="AL5809"/>
+<part name="D4" library="diode" deviceset="DIODE-" device="SOD123" value="AL5809"/>
 <part name="D1" library="diode" deviceset="DIODE-" device="SOD123" value="AL5809"/>
 <part name="D2" library="diode" deviceset="DIODE-" device="SOD123" value="AL5809"/>
 <part name="JP2" library="SparkFun-Connectors" deviceset="M01" device="PTH"/>
+<part name="FRAME1" library="SparkFun-Aesthetics" deviceset="FRAME-LETTER" device=""/>
 </parts>
 <sheets>
 <sheet>
 <plain>
+<text x="104.14" y="-167.64" size="1.778" layer="94">Chris Kelley</text>
 </plain>
 <instances>
@@
 <instance part="LED3" gate="G$1" x="22.86" y="-78.74"/>
 <instance part="LED4" gate="G$1" x="22.86" y="-106.68"/>
-<instance part="U$3" gate="G$1" x="30.48" y="-147.32" rot="R90"/>
+<instance part="S1" gate="G$1" x="30.48" y="-147.32" rot="R90"/>
 <instance part="C2" gate="G$1" x="22.86" y="-157.48" rot="R90"/>
-<instance part="JP1" gate="G$1" x="91.44" y="-78.74" rot="R180"/>
+<instance part="HS1" gate="G$1" x="91.44" y="-78.74" rot="R180"/>
 <instance part="JP5" gate="G$1" x="60.96" y="-76.2" rot="R180"/>
 <instance part="JP6" gate="G$1" x="60.96" y="-88.9" rot="R180"/>
 <instance part="GND1" gate="1" x="81.28" y="-88.9"/>
-<instance part="D5" gate="G$1" x="0" y="-20.32"/>
-<instance part="D6" gate="G$1" x="0" y="-48.26"/>
+<instance part="D3" gate="G$1" x="0" y="-20.32"/>
+<instance part="D4" gate="G$1" x="0" y="-48.26"/>
 <instance part="D1" gate="G$1" x="-2.54" y="-73.66"/>
 <instance part="D2" gate="G$1" x="-2.54" y="-101.6"/>
 <instance part="JP2" gate="G$1" x="60.96" y="-101.6" rot="R180"/>
+<instance part="FRAME1" gate="G$1" x="-71.12" y="-177.8"/>
+<instance part="FRAME1" gate="V" x="76.2" y="-177.8"/>
 </instances>
 <busses>
@@
 </segment>
 <segment>
-<pinref part="U$3" gate="G$1" pin="GND"/>
+<pinref part="S1" gate="G$1" pin="GND"/>
 <wire x1="-2.54" y1="-144.78" x2="5.08" y2="-144.78" width="0.1524" layer="91"/>
 <label x="-2.54" y="-144.78" size="1.778" layer="95"/>
@@
 </segment>
 <segment>
-<pinref part="U$3" gate="G$1" pin="S3"/>
+<pinref part="S1" gate="G$1" pin="S3"/>
 <wire x1="48.26" y1="-129.54" x2="35.56" y2="-129.54" width="0.1524" layer="91"/>
 <label x="43.18" y="-129.54" size="1.778" layer="95"/>
@@
 </segment>
 <segment>
-<pinref part="JP1" gate="G$1" pin="6"/>
+<pinref part="HS1" gate="G$1" pin="6"/>
 <wire x1="78.74" y1="-86.36" x2="81.28" y2="-86.36" width="0.1524" layer="91"/>
 <pinref part="GND1" gate="1" pin="GND"/>
@@
 </segment>
 <segment>
-<pinref part="U$3" gate="G$1" pin="OUT"/>
+<pinref part="S1" gate="G$1" pin="OUT"/>
 <wire x1="48.26" y1="-139.7" x2="35.56" y2="-139.7" width="0.1524" layer="91"/>
 <label x="43.18" y="-139.7" size="1.778" layer="95"/>
@@
 <segment>
 <wire x1="-10.16" y1="-20.32" x2="-2.54" y2="-20.32" width="0.1524" layer="91"/>
-<pinref part="D5" gate="G$1" pin="A"/>
+<pinref part="D3" gate="G$1" pin="A"/>
 <label x="-10.16" y="-20.32" size="1.778" layer="95"/>
 </segment>
@@
 <net name="PC1_2" class="0">
 <segment>
-<pinref part="U$3" gate="G$1" pin="OE"/>
+<pinref part="S1" gate="G$1" pin="OE"/>
 <wire x1="-2.54" y1="-139.7" x2="10.16" y2="-139.7" width="0.1524" layer="91"/>
 <label x="-2.54" y="-139.7" size="1.778" layer="95"/>
 </segment>
 <segment>
-<pinref part="JP1" gate="G$1" pin="5"/>
+<pinref part="HS1" gate="G$1" pin="5"/>
 <wire x1="78.74" y1="-83.82" x2="86.36" y2="-83.82" width="0.1524" layer="91"/>
 <label x="73.66" y="-83.82" size="1.778" layer="95"/>
@@
 <net name="VCC_2" class="0">
 <segment>
-<pinref part="U$3" gate="G$1" pin="S2"/>
+<pinref part="S1" gate="G$1" pin="S2"/>
 <wire x1="48.26" y1="-134.62" x2="35.56" y2="-134.62" width="0.1524" layer="91"/>
 <label x="43.18" y="-134.62" size="1.778" layer="95"/>
 </segment>
 <segment>
-<pinref part="U$3" gate="G$1" pin="VDD"/>
+<pinref part="S1" gate="G$1" pin="VDD"/>
 <wire x1="48.26" y1="-144.78" x2="40.64" y2="-144.78" width="0.1524" layer="91"/>
 <label x="43.18" y="-144.78" size="1.778" layer="95"/>
@@
 </segment>
 <segment>
-<pinref part="JP1" gate="G$1" pin="4"/>
+<pinref part="HS1" gate="G$1" pin="4"/>
 <wire x1="81.28" y1="-81.28" x2="86.36" y2="-81.28" width="0.1524" layer="91"/>
 <wire x1="78.74" y1="-81.28" x2="81.28" y2="-81.28" width="0.1524" layer="91"/>
@@
 </segment>
 <segment>
-<pinref part="U$3" gate="G$1" pin="S0"/>
+<pinref part="S1" gate="G$1" pin="S0"/>
 <wire x1="-2.54" y1="-129.54" x2="10.16" y2="-129.54" width="0.1524" layer="91"/>
 <label x="-2.54" y="-129.54" size="1.778" layer="95"/>
@@
 </segment>
 <segment>
-<pinref part="D6" gate="G$1" pin="A"/>
+<pinref part="D4" gate="G$1" pin="A"/>
 <wire x1="-2.54" y1="-48.26" x2="-10.16" y2="-48.26" width="0.1524" layer="91"/>
 <label x="-10.16" y="-48.26" size="1.778" layer="95"/>
@@
 <net name="N$7" class="0">
 <segment>
-<pinref part="D5" gate="G$1" pin="C"/>
+<pinref part="D3" gate="G$1" pin="C"/>
 <pinref part="LED2" gate="G$1" pin="A"/>
 <wire x1="22.86" y1="-20.32" x2="22.86" y2="-22.86" width="0.1524" layer="91"/>
@@
 <net name="N$5" class="0">
 <segment>
-<pinref part="D6" gate="G$1" pin="C"/>
+<pinref part="D4" gate="G$1" pin="C"/>
 <pinref part="LED1" gate="G$1" pin="A"/>
 <wire x1="22.86" y1="-48.26" x2="22.86" y2="-50.8" width="0.1524" layer="91"/>
@@
 </segment>
 <segment>
-<pinref part="U$3" gate="G$1" pin="S1"/>
+<pinref part="S1" gate="G$1" pin="S1"/>
 <wire x1="-2.54" y1="-134.62" x2="10.16" y2="-134.62" width="0.1524" layer="91"/>
 <label x="-2.54" y="-134.62" size="1.778" layer="95"/>
